Commit message: added realsense

File: urdf/ty_sensor_mount.xacro (robot description, xacro)
@@ -5,4 +5,6 @@
 <xacro:include filename="$(find ty_sensor_mount)/gazebo/ty_sensor_mount_physics.gazebo" />
 <xacro:include filename="$(find ty_sensor_mount)/gazebo/ty_sensor_mount_plugins.gazebo" />
+<xacro:include filename="$(find realsense)/urdf/realsense.urdf.xacro" />
+<xacro:include filename="$(find realsense_ros_gazebo)/xacro/tracker.xacro"/>
 <link name="world"/>
 <link name="sensor_mount_base">
@@ -66,4 +68,12 @@
   </collision>
 </link>
+<!--#####################  REALSENSE  ##########################-->
+<realsense parent="sensor_mount_base">
+  <origin xyz="-0.0025 0 0.1125" rpy="0 0 0"/>
+</realsense>
+<xacro:realsense_T265 sensor_name="camera" parent_link="sensor_mount_base" rate="30.0">
+  <origin rpy="0 0 0" xyz="0.00625 0 0.0875"/>
+</xacro:realsense_T265>
+<!--#####################  JOINTS  ##########################-->
 <joint name="world_joint" type="fixed">
   <origin rpy="0 0 0" xyz="0.02 0 0"/>

Commit message: added new realsense

File: urdf/ty_sensor_mount.xacro (robot description, xacro)
@@ -5,6 +5,6 @@
 <xacro:include filename="$(find ty_sensor_mount)/gazebo/ty_sensor_mount_physics.gazebo" />
 <xacro:include filename="$(find ty_sensor_mount)/gazebo/ty_sensor_mount_plugins.gazebo" />
-<xacro:include filename="$(find realsense)/urdf/realsense.urdf.xacro" />
 <xacro:include filename="$(find realsense_ros_gazebo)/xacro/tracker.xacro"/>
+<xacro:include filename="$(find realsense_ros_gazebo)/xacro/depthcam.xacro"/>
 <link name="world"/>
 <link name="sensor_mount_base">
@@ -69,10 +69,10 @@
 </link>
 <!--#####################  REALSENSE  ##########################-->
-<realsense parent="sensor_mount_base">
-  <origin xyz="-0.0025 0 0.1125" rpy="0 0 0"/>
-</realsense>
 <xacro:realsense_T265 sensor_name="camera" parent_link="sensor_mount_base" rate="30.0">
   <origin rpy="0 0 0" xyz="0.00625 0 0.0875"/>
 </xacro:realsense_T265>
+<xacro:realsense_d435 sensor_name="d435" parent_link="sensor_mount_base" rate="10">
+  <origin rpy="0 0 0" xyz="-0.0025 0 0.1125"/>
+</xacro:realsense_d435>
 <!--#####################  JOINTS  ##########################-->
 <joint name="world_joint" type="fixed">
