Commit message: added macro to attach to different robots

File: urdf/materials.xacro (robot description, xacro)
@@ -1,5 +1,5 @@
 <?xml version="1.0" ?>
 <robot name="ty_sensor_mount" xmlns:xacro="http://www.ros.org/wiki/xacro" >
-<material name="silver">
+<material name="ty_color">
   <color rgba="0.700 0.700 0.700 1.000"/>
 </material>

File: urdf/ty_sensor_mount.xacro (robot description, xacro)
@@ -7,5 +7,5 @@
 <xacro:include filename="$(find realsense_ros_gazebo)/xacro/tracker.xacro"/>
 <xacro:include filename="$(find realsense_ros_gazebo)/xacro/depthcam.xacro"/>
-<link name="world"/>
+<xacro:macro name="ty_sensor" params="name:=ty_sensor parent *origin">
 <link name="sensor_mount_base">
   <inertial>
@@ -19,5 +19,5 @@
       <mesh filename="package://ty_sensor_mount/meshes/sensor_mount_base.stl" scale="0.001 0.001 0.001"/>
     </geometry>
-    <material name="silver"/>
+    <material name="ty_color"/>
   </visual>
   <collision>
@@ -39,5 +39,5 @@
       <mesh filename="package://ty_sensor_mount/meshes/lidar_base.stl" scale="0.001 0.001 0.001"/>
     </geometry>
-    <material name="silver"/>
+    <material name="ty_color"/>
   </visual>
   <collision>
@@ -59,5 +59,5 @@
       <mesh filename="package://ty_sensor_mount/meshes/lidar.stl" scale="0.001 0.001 0.001"/>
     </geometry>
-    <material name="silver"/>
+    <material name="ty_color"/>
   </visual>
   <collision>
@@ -76,8 +76,15 @@
 </xacro:realsense_d435>
 <!--#####################  JOINTS  ##########################-->
+<!--
 <joint name="world_joint" type="fixed">
   <origin rpy="0 0 0" xyz="0.02 0 0"/>
   <parent link="world"/>
   <child link="sensor_mount_base"/>
+</joint>
+-->
+<joint name="${name}_joint" type="fixed">
+  <xacro:insert_block name="origin" />
+  <parent link="${parent}"/>
+  <child link="sensor_mount_base" />
 </joint>
 <joint name="Rigid1" type="fixed">
@@ -91,3 +98,4 @@
   <child link="lidar"/>
 </joint>
+</xacro:macro>
 </robot>
